Commit message: Adds box as collision geometry.

File: tams_ur5_description/urdf/s_model_adapter.urdf.xacro (robot description, xacro)
@@ -36,4 +36,10 @@
         </geometry>
       </collision>
+      <collision>
+        <origin xyz="0.0725 0 0" rpy="0 0 0.0" />
+        <geometry>
+	  <box size="0.035 0.035 0.035"/>
+        </geometry>
+      </collision>
     </link>
     <joint name="${name}_joint" type="fixed">
