Commit message: Update plug collision model for wireless gripper

File: tams_ur5_description/urdf/plug_collision_model.urdf.xacro (robot description, xacro)
@@ -14,7 +14,7 @@
       </inertial>
       <collision>
-        <origin xyz="0.0855 0.065 0.0" rpy="0.0 0.0 0.0" />
+        <origin xyz="0.08 -0.05 0.0" rpy="0.0 0.0 0.0" />
         <geometry>
-          <box size="0.05 0.10 0.075"/>
+          <box size="0.08 0.10 0.075"/>
         </geometry>
       </collision>
@@ -36,7 +36,7 @@
       </inertial>
       <collision>
-        <origin xyz="0.025 -0.01 0.09" rpy="0.0 0.0 0.0" />
+        <origin xyz="0.025 -0.025 0.06" rpy="0.0 0.0 0.0" />
         <geometry>
-          <box size="0.03 0.06 0.06"/>
+          <box size="0.03 0.09 0.12"/>
         </geometry>
       </collision>
