Commit message: update tams_ur5 robot description file ur5.urdf.xacro

File: tams_ur5_description/urdf/ur5.urdf.xacro (robot description, xacro)
@@ -79,5 +79,7 @@
     https://github.com/Xamla/xamla_egomo/tree/master/egomo_3d_printed_parts/egomo-1
   -->
-  <xacro:macro name="ur5_robot" params="prefix joint_limited xamla_cap:=false">
+  <xacro:macro name="ur5_robot" params="prefix joint_limited
+    xamla_cap:=false
+    transmission_hw_interface:=hardware_interface/PositionJointInterface">
     <link name="${prefix}base_link" >
       <visual>
@@ -307,5 +309,5 @@
       </collision>
     </link>
-    <xacro:ur_arm_transmission prefix="${prefix}" />
+    <xacro:ur_arm_transmission prefix="${prefix}" hw_interface="${transmission_hw_interface}" />
     <xacro:ur_arm_gazebo prefix="${prefix}" />
     <!-- ROS base_link to UR 'Base' Coordinates transform -->
