Commit message: add pi as a constant variable

File: tams_ur5_description/urdf/arm.urdf.xacro (robot description, xacro)
@@ -2,4 +2,5 @@
 <robot xmlns:xacro="http://www.ros.org/wiki/xacro"
        name="arm" >
+  <xacro:property name="pi" value="3.1415926535897931" />
   <!-- include macro definitions -->
   <xacro:include filename="$(find ur_description)/urdf/gazebo.urdf.xacro" />
@@ -11,5 +12,5 @@
   <xacro:ur5_robot prefix="" joint_limited="true"/>
   <xacro:robotiq_fts150 prefix="ft_" parent="ee_link">
-    <origin xyz="0.0 0.0 0.012" rpy="0.0 1.571 0.0" />
+    <origin xyz="0.0 0.0 0.012" rpy="0.0 ${pi/2} 0.0" />
   </xacro:robotiq_fts150>
   <!-- the adaptive gripper -->
@@ -18,5 +19,5 @@
     <parent link="ft_fts_toolside" />
     <child link = "palm" />
-    <origin xyz="0.0 0.0 0.06" rpy="1.57079632679 0.0 1.570797" />
+    <origin xyz="0.0 0.0 0.06" rpy="${pi/2} 0.0 ${pi/2}" />
   </joint>
 </robot>

Commit message: Set prefix due to insertion of tool0 from robotiqs gripper
in the last update of robotiqs s model gripper the tooframe tool0 was
merged. The ur5 has also a tool0 so we have to set a prefix for the
gripper.

File: tams_ur5_description/urdf/arm.urdf.xacro (robot description, xacro)
@@ -14,8 +14,8 @@
   </xacro:robotiq_fts150>
   <!-- the adaptive gripper -->
-  <xacro:s-model_articulated prefix=""/>
+  <xacro:s-model_articulated prefix="s_model_"/>
   <joint name="gripper_joint" type="fixed">
     <parent link="ft_fts_toolside" />
-    <child link = "palm" />
+    <child link = "s_model_palm" />
     <origin xyz="0.0 0.0 0.06" rpy="${pi/2} 0.0 ${pi/2}" />
   </joint>

Commit message: Corrected positioning of ft-sensor in urdf
The origin of the force torque sensor was set to 1.2 cm in z direction
of the ee_link, due to the assumption that the z-axis shows in the
direkten of the ft sensor/gripper. This assumption was wrong, the x-axis
of the ee_link ponts in this direction, so this was changed.
The second change is the value. In the urdf file it is described that
the adapter is 9mm height instead of 12mm. When we measure it, 9mm fits
better then 12mm.
The rotation of the force torque sensor was changed, now the connection
points into the right direction. Due to that the rotation of the gripper
had to be fixed too.

File: tams_ur5_description/urdf/arm.urdf.xacro (robot description, xacro)
@@ -11,5 +11,5 @@
   <xacro:ur5_robot prefix="" joint_limited="true"/>
   <xacro:robotiq_fts150 prefix="ft_" parent="ee_link">
-    <origin xyz="0.0 0.0 0.012" rpy="0.0 ${pi/2} 0.0" />
+    <origin xyz="0.009 0.0 0.0" rpy="0.0 ${-pi/2} ${pi}" />
   </xacro:robotiq_fts150>
   <!-- the adaptive gripper -->
@@ -18,5 +18,5 @@
     <parent link="ft_fts_toolside" />
     <child link = "s_model_palm" />
-    <origin xyz="0.0 0.0 0.06" rpy="${pi/2} 0.0 ${pi/2}" />
+    <origin xyz="0.0 0.0 0.06" rpy="${pi/2} 0.0 ${-pi/2}" />
   </joint>
 </robot>

Commit message: New adapter models for ft sensor and gripper
Createt new adapter xacros to complete the urdf for our arm.
The position of the gripper was decresed by -3mm in z direction.(in
direction of the ft sensor) due to measuring errors.

File: tams_ur5_description/urdf/arm.urdf.xacro (robot description, xacro)
@@ -6,11 +6,26 @@
   <xacro:include filename="$(find ur_description)/urdf/ur5.urdf.xacro" />
   <xacro:include filename="$(find robotiq_s_model_visualization)/cfg/s-model_articulated_macro.xacro" />
-  <!-- ft150 -->
   <xacro:include filename="$(find robotiq_force_torque_sensor)/urdf/robotiq_fts150.urdf.xacro" />
+  <xacro:include filename="$(find tams_ur5_description)/urdf/ft_adapter.urdf.xacro" />
+  <xacro:include filename="$(find tams_ur5_description)/urdf/s_model_adapter.urdf.xacro" />
   <!-- arm -->
   <xacro:ur5_robot prefix="" joint_limited="true"/>
+  <!-- ft_adapter -->
+  <joint name="ft_adapter" type="fixed">
+    <parent link="ee_link" />
+    <child link = "ft_adapter" />
+    <origin xyz="0.0045 0.0 0.0" rpy="0.0 ${pi/2} 0.0" />
+  </joint>
+  <xacro:ft_adapter name="ft_adapter" parent="ee_link">
+    <origin xyz="0.0045 0.0 0.0" rpy="0.0 ${pi/2} 0.0" />
+  </xacro:ft_adapter>
+  <!-- ft150 -->
   <xacro:robotiq_fts150 prefix="ft_" parent="ee_link">
     <origin xyz="0.009 0.0 0.0" rpy="0.0 ${-pi/2} ${pi}" />
   </xacro:robotiq_fts150>
+  <!-- s_model_adapter -->
+  <xacro:s_model_adapter name="s_model_adapter" parent="ft_fts_toolside">
+    <origin xyz="0.0 0.0 0.0065" rpy="0.0 0.0 0.0" />
+  </xacro:s_model_adapter>
   <!-- the adaptive gripper -->
   <xacro:s-model_articulated prefix="s_model_"/>
@@ -18,5 +33,5 @@
     <parent link="ft_fts_toolside" />
     <child link = "s_model_palm" />
-    <origin xyz="0.0 0.0 0.06" rpy="${pi/2} 0.0 ${-pi/2}" />
+    <origin xyz="0.0 0.0 0.057" rpy="${pi/2} 0.0 ${-pi/2}" />
   </joint>
 </robot>

Commit message: new link tool0 and prefix for ur5
We want to use pick and place, in this case we noticed that the ee_link
has another orientation as the eef of the gripper, so we inserted a new
link tool0 at the origin of the fts_toolside with the same orientation
as the s_model_tool_0. The ur5 has already a tool0, so we set a prefix
for the ur5.
The new tool0 link is the eef of the ur5 now.

File: tams_ur5_description/urdf/arm.urdf.xacro (robot description, xacro)
@@ -10,18 +10,25 @@
   <xacro:include filename="$(find tams_ur5_description)/urdf/s_model_adapter.urdf.xacro" />
   <!-- arm -->
-  <xacro:ur5_robot prefix="" joint_limited="true"/>
+  <xacro:ur5_robot prefix="ur5_" joint_limited="true"/>
   <!-- ft_adapter -->
   <joint name="ft_adapter" type="fixed">
-    <parent link="ee_link" />
+    <parent link="ur5_ee_link" />
     <child link = "ft_adapter" />
     <origin xyz="0.0045 0.0 0.0" rpy="0.0 ${pi/2} 0.0" />
   </joint>
-  <xacro:ft_adapter name="ft_adapter" parent="ee_link">
+  <xacro:ft_adapter name="ft_adapter" parent="ur5_ee_link">
     <origin xyz="0.0045 0.0 0.0" rpy="0.0 ${pi/2} 0.0" />
   </xacro:ft_adapter>
   <!-- ft150 -->
-  <xacro:robotiq_fts150 prefix="ft_" parent="ee_link">
+  <xacro:robotiq_fts150 prefix="ft_" parent="ur5_ee_link">
     <origin xyz="0.009 0.0 0.0" rpy="0.0 ${-pi/2} ${pi}" />
   </xacro:robotiq_fts150>
+  <!-- tool0 frame -->
+  <link name="tool0" />
+  <joint name="ft_fts_toolside_tool0" type="fixed">
+    <parent link="ft_fts_toolside"/>
+    <child link="tool0"/>
+    <origin xyz="0.0 0.0 0.0" rpy="0.0 ${-pi/2} 0.0"/>
+  </joint>
   <!-- s_model_adapter -->
   <xacro:s_model_adapter name="s_model_adapter" parent="ft_fts_toolside">
@@ -31,7 +38,7 @@
   <xacro:s-model_articulated prefix="s_model_"/>
   <joint name="gripper_joint" type="fixed">
-    <parent link="ft_fts_toolside" />
+    <parent link="tool0" />
     <child link = "s_model_palm" />
-    <origin xyz="0.0 0.0 0.057" rpy="${pi/2} 0.0 ${-pi/2}" />
+    <origin xyz="0.057 0.0 0.0" rpy="0.0 0.0 ${-pi/2}" />
   </joint>
 </robot>

Commit message: Collision models for gripper and ft plugs
The plugs of the gripper and the ft sensor have collision models now.
Due to the use of pick, the self collisions are often very close, so we decided to model the plugs.

File: tams_ur5_description/urdf/arm.urdf.xacro (robot description, xacro)
@@ -9,4 +9,5 @@
   <xacro:include filename="$(find tams_ur5_description)/urdf/ft_adapter.urdf.xacro" />
   <xacro:include filename="$(find tams_ur5_description)/urdf/s_model_adapter.urdf.xacro" />
+  <xacro:include filename="$(find tams_ur5_description)/urdf/plug_collision_model.urdf.xacro" />
   <!-- arm -->
   <xacro:ur5_robot prefix="ur5_" joint_limited="true"/>
@@ -42,3 +43,7 @@
     <origin xyz="0.057 0.0 0.0" rpy="0.0 0.0 ${-pi/2}" />
   </joint>
+  <!-- plug collision model -->
+  <xacro:plug_collision_model name="plug_collision_model" parent="ur5_ee_link" >
+    <origin xyz="0.0 0.0 0.0" rpy="0.0 0.0 0.0" />
+  </xacro:plug_collision_model>
 </robot>

Commit message: remove redundant joint from arm urdf

File: tams_ur5_description/urdf/arm.urdf.xacro (robot description, xacro)
@@ -13,9 +13,4 @@
   <xacro:ur5_robot prefix="ur5_" joint_limited="true"/>
   <!-- ft_adapter -->
-  <joint name="ft_adapter" type="fixed">
-    <parent link="ur5_ee_link" />
-    <child link = "ft_adapter" />
-    <origin xyz="0.0045 0.0 0.0" rpy="0.0 ${pi/2} 0.0" />
-  </joint>
   <xacro:ft_adapter name="ft_adapter" parent="ur5_ee_link">
     <origin xyz="0.0045 0.0 0.0" rpy="0.0 ${pi/2} 0.0" />

Commit message: Changes gripper adapter to wireles custom version.

File: tams_ur5_description/urdf/arm.urdf.xacro (robot description, xacro)
@@ -31,5 +31,5 @@
   <!-- s_model_adapter -->
   <xacro:s_model_adapter name="s_model_adapter" parent="ft_fts_toolside">
-    <origin xyz="0.0 0.0 0.0065" rpy="0.0 0.0 0.0" />
+    <origin xyz="0.0 0.0 0.015" rpy="0.0 0.0 0.0" />
   </xacro:s_model_adapter>
   <!-- the adaptive gripper -->
@@ -38,5 +38,5 @@
     <parent link="tool0" />
     <child link = "s_model_palm" />
-    <origin xyz="0.057 0.0 0.0" rpy="0.0 0.0 ${-pi/2}" />
+    <origin xyz="0.0775 0.0 0.0" rpy="0.0 0.0 ${-pi/2}" />
   </joint>
   <!-- plug collision model -->

File: tams_ur5_description/urdf/s_model_adapter.urdf.xacro (robot description, xacro)
@@ -15,5 +15,14 @@
         <origin xyz="0.0 0 0.0" rpy="0 0 0.0" />
         <geometry>
-          <cylinder length="0.013" radius="0.04"/>
+ 	  <cylinder length="0.035" radius="0.06"/>
+        </geometry>
+        <material name="gray">
+          <color rgba="0.2 0.2 0.2 1"/>
+        </material>
+      </visual>
+      <visual>
+        <origin xyz="0.0725 0 0" rpy="0 0 0.0" />
+        <geometry>
+	  <box size="0.035 0.035 0.035"/>
         </geometry>
         <material name="gray">
@@ -24,5 +33,5 @@
         <origin xyz="0.0 0 0.0" rpy="0 0 0.0" />
         <geometry>
-          <cylinder length="0.013" radius="0.04"/>
+          <cylinder length="0.035" radius="0.06"/>
         </geometry>
       </collision>

Commit message: Fixes gripper palm orientation. Adjusts plug collision models. Removes whitespace.

File: tams_ur5_description/urdf/arm.urdf.xacro (robot description, xacro)
@@ -27,5 +27,5 @@
     <parent link="ft_fts_toolside"/>
     <child link="tool0"/>
-    <origin xyz="0.0 0.0 0.0" rpy="0.0 ${-pi/2} 0.0"/>
+    <origin xyz="0.0 0.0 0.0205" rpy="0.0 ${-pi/2} 0.0"/>
   </joint>
   <!-- s_model_adapter -->
@@ -38,5 +38,5 @@
     <parent link="tool0" />
     <child link = "s_model_palm" />
-    <origin xyz="0.0775 0.0 0.0" rpy="0.0 0.0 ${-pi/2}" />
+    <origin xyz="0.057 0.0 0.0" rpy="0.0 ${pi} ${-pi/2}" />
   </joint>
   <!-- plug collision model -->

File: tams_ur5_description/urdf/plug_collision_model.urdf.xacro (robot description, xacro)
@@ -14,5 +14,5 @@
       </inertial>
       <collision>
-        <origin xyz="0.065 0.065 0.0" rpy="0.0 0.0 0.0" />
+        <origin xyz="0.0855 0.065 0.0" rpy="0.0 0.0 0.0" />
         <geometry>
           <box size="0.05 0.10 0.075"/>

Commit message: Added sim parameter and inorder parameter to launch files

File: tams_ur5_description/urdf/arm.urdf.xacro (robot description, xacro)
@@ -4,43 +4,65 @@
   <xacro:property name="pi" value="3.1415926535897931" />
   <!-- include macro definitions -->
+  <!-- common stuff (ros_control gazebo) -->
+  <xacro:include filename="$(find ur_description)/urdf/common.gazebo.xacro" />
   <xacro:include filename="$(find ur_description)/urdf/ur5.urdf.xacro" />
   <xacro:include filename="$(find robotiq_s_model_visualization)/cfg/s-model_articulated_macro.xacro" />
+  <xacro:include filename="$(find robotiq_s_model_visualization)/cfg/robotiq_hand_macro.urdf.xacro" />
   <xacro:include filename="$(find robotiq_force_torque_sensor)/urdf/robotiq_fts150.urdf.xacro" />
   <xacro:include filename="$(find tams_ur5_description)/urdf/ft_adapter.urdf.xacro" />
   <xacro:include filename="$(find tams_ur5_description)/urdf/s_model_adapter.urdf.xacro" />
   <xacro:include filename="$(find tams_ur5_description)/urdf/plug_collision_model.urdf.xacro" />
-  <!-- arm -->
-  <!-- xamla_cap is a custom parameter in TAMS' fork of the universal_robot repository,
-       remove it if you want to use the upstream ur5 description instead -->
-  <xacro:ur5_robot prefix="ur5_" joint_limited="true" xamla_cap="true"/>
-  <!-- ft_adapter -->
-  <xacro:ft_adapter name="ft_adapter" parent="ur5_ee_link">
-    <origin xyz="0.0045 0.0 0.0" rpy="0.0 ${pi/2} 0.0" />
-  </xacro:ft_adapter>
-  <!-- ft150 -->
-  <xacro:robotiq_fts150 prefix="ft_" parent="ur5_ee_link">
-    <origin xyz="0.009 0.0 0.0" rpy="0.0 ${-pi/2} ${pi}" />
-  </xacro:robotiq_fts150>
-  <!-- tool0 frame -->
-  <link name="tool0" />
-  <joint name="ft_fts_toolside_tool0" type="fixed">
-    <parent link="ft_fts_toolside"/>
-    <child link="tool0"/>
-    <origin xyz="0.0 0.0 0.0205" rpy="0.0 ${-pi/2} 0.0"/>
-  </joint>
-  <!-- s_model_adapter -->
-  <xacro:s_model_adapter name="s_model_adapter" parent="ft_fts_toolside">
-    <origin xyz="0.0 0.0 0.015" rpy="0.0 0.0 0.0" />
-  </xacro:s_model_adapter>
-  <!-- the adaptive gripper -->
-  <xacro:s-model_articulated prefix="s_model_"/>
-  <joint name="gripper_joint" type="fixed">
-    <parent link="tool0" />
-    <child link = "s_model_palm" />
-    <origin xyz="0.057 0.0 0.0" rpy="0.0 ${pi} ${-pi/2}" />
-  </joint>
-  <!-- plug collision model -->
-  <xacro:plug_collision_model name="plug_collision_model" parent="ur5_ee_link" >
-    <origin xyz="0.0 0.0 0.0" rpy="0.0 0.0 0.0" />
-  </xacro:plug_collision_model>
+  <xacro:macro name="arm" params="sim">
+    <!-- arm -->
+    <!-- xamla_cap is a custom parameter in TAMS' fork of the universal_robot repository,
+         remove it if you want to use the upstream ur5 description instead -->
+    <xacro:ur5_robot prefix="ur5_" joint_limited="true" xamla_cap="true"/>
+    <!-- ft_adapter -->
+    <xacro:ft_adapter name="ft_adapter" parent="ur5_ee_link">
+      <origin xyz="0.0045 0.0 0.0" rpy="0.0 ${pi/2} 0.0" />
+    </xacro:ft_adapter>
+    <!-- ft150 -->
+    <xacro:robotiq_fts150 prefix="ft_" parent="ur5_ee_link">
+      <origin xyz="0.009 0.0 0.0" rpy="0.0 ${-pi/2} ${pi}" />
+    </xacro:robotiq_fts150>
+    <!-- tool0 frame -->
+    <link name="tool0" />
+    <joint name="ft_fts_toolside_tool0" type="fixed">
+      <parent link="ft_fts_toolside"/>
+      <child link="tool0"/>
+      <origin xyz="0.0 0.0 0.0205" rpy="0.0 ${-pi/2} 0.0"/>
+    </joint>
+    <!-- s_model_adapter -->
+    <xacro:s_model_adapter name="s_model_adapter" parent="ft_fts_toolside">
+      <origin xyz="0.0 0.0 0.015" rpy="0.0 0.0 0.0" />
+    </xacro:s_model_adapter>
+    <!-- the adaptive gripper -->
+    <!-- real world, may be deprecated later on-->
+    <xacro:unless value="${sim}">
+      <xacro:s-model_articulated prefix="s_model_"/>
+      <joint name="gripper_joint" type="fixed">
+        <parent link="tool0" />
+        <child link="s_model_palm" />
+        <origin xyz="0.057 0.0 0.0" rpy="0.0 ${pi} ${-pi/2}" />
+      </joint>
+    </xacro:unless>
+    <!-- gazebo -->
+    <xacro:if value="${sim}">
+      <xacro:robotiq_hand prefix="s_model_" reflect="" parent="tool0">
+        <origin xyz="0.057 0.0 0.0" rpy="0.0 ${pi} ${-pi/2}" />
+      </xacro:robotiq_hand>
+      <gazebo>
+        <plugin name="robotiq_plugin" filename="libRobotiqHandPlugin.so">
+          <!--<side>s_model_</side>-->
+          <prefix>s_model_</prefix>#
+          <kp_position>5.0</kp_position>
+          <kd_position>0.5</kd_position>
+        </plugin>
+      </gazebo>
+    </xacro:if>
+    <!-- plug collision model -->
+    <xacro:plug_collision_model name="plug_collision_model" parent="ur5_ee_link" >
+      <origin xyz="0.0 0.0 0.0" rpy="0.0 0.0 0.0" />
+    </xacro:plug_collision_model>
+  </xacro:macro>
 </robot>

Commit message: add camera holder link and r200_camera_link
4 new models in mesh folder, and an argument for using r200

File: tams_ur5_description/urdf/arm.urdf.xacro (robot description, xacro)
@@ -2,4 +2,5 @@
 <robot xmlns:xacro="http://www.ros.org/wiki/xacro"
        name="arm" >
+  <xacro:arg name="r200" default="true" />
   <xacro:property name="pi" value="3.1415926535897931" />
   <!-- include macro definitions -->
@@ -10,4 +11,5 @@
   <xacro:include filename="$(find tams_ur5_description)/urdf/s_model_adapter.urdf.xacro" />
   <xacro:include filename="$(find tams_ur5_description)/urdf/plug_collision_model.urdf.xacro" />
+  <xacro:include filename="$(find tams_ur5_description)/urdf/mounted_camera.urdf.xacro" />
   <!-- arm -->
   <!-- xamla_cap is a custom parameter in TAMS' fork of the universal_robot repository,
@@ -18,4 +20,10 @@
     <origin xyz="0.0045 0.0 0.0" rpy="0.0 ${pi/2} 0.0" />
   </xacro:ft_adapter>
+  <!-- mounted_camera -->
+  <xacro:if value="$(arg r200)">
+    <xacro:mounted_camera name="mounted_camera" parent="ft_adapter">
+        <origin xyz="0 0 0.0" rpy="0 0 0" />
+    </xacro:mounted_camera>
+  </xacro:if>
   <!-- ft150 -->
   <xacro:robotiq_fts150 prefix="ft_" parent="ur5_ee_link">

Commit message: remove definition of pi as it already predefined

File: tams_ur5_description/urdf/arm.urdf.xacro (robot description, xacro)
@@ -3,5 +3,4 @@
        name="arm" >
   <xacro:arg name="r200" default="true" />
-  <xacro:property name="pi" value="3.1415926535897931" />
   <!-- include macro definitions -->
   <xacro:include filename="$(find tams_ur5_description)/urdf/ur5.urdf.xacro" />

File: tams_ur5_description/urdf/ur5.urdf.xacro (robot description, xacro)
@@ -3,5 +3,4 @@
   <xacro:include filename="$(find ur_description)/urdf/ur.transmission.xacro" />
   <xacro:include filename="$(find ur_description)/urdf/ur.gazebo.xacro" />
-  <xacro:property name="pi" value="3.14159265" />
   <!-- Inertia parameters -->
   <xacro:property name="base_mass" value="4.0" />  <!-- This mass might be incorrect -->
